Commit message: heros robot addad

File: bresilla/urdf/bresilla.xacro (robot description, xacro)
@@ -1,5 +1,5 @@
 <?xml version='1.0'?>
-<robot name="rover" xmlns:xacro="http://www.ros.org/wiki/xacro">
-    <xacro:include filename="$(find rover)/urdf/rover.gazebo" />
+<robot name="bresilla" xmlns:xacro="http://www.ros.org/wiki/xacro">
+    <xacro:include filename="$(find bresilla)/urdf/bresilla.gazebo" />
     <link name="robot_footprint"></link>
     <joint name="robot_footprint_joint" type="fixed">
@@ -101,5 +101,5 @@
             <origin xyz="0.0 0 0" rpy=" 0 0 0"/>
             <geometry>
-                <mesh filename="package://rover/meshes/hokuyo.dae"/>
+                <mesh filename="package://bresilla/meshes/hokuyo.dae"/>
                 <!-- <box size="0.1 0.1 0.1"/> -->
             </geometry>

Commit message: robot finished, just parameter tuning left

File: bresilla/urdf/bresilla.xacro (robot description, xacro)
@@ -1,6 +1,24 @@
 <?xml version='1.0'?>
 <robot name="bresilla" xmlns:xacro="http://www.ros.org/wiki/xacro">
-    <xacro:include filename="$(find bresilla)/urdf/bresilla.gazebo" />
+    <xacro:include filename="$(find bresilla)/urdf/sensors/camera.xacro" />
+    <xacro:include filename="$(find bresilla)/urdf/sensors/hokuyo.xacro" />
     <link name="robot_footprint"></link>
+    <gazebo>
+        <plugin name="differential_drive_controller" filename="libgazebo_ros_diff_drive.so">
+            <legacyMode>false</legacyMode>
+            <alwaysOn>true</alwaysOn>
+            <updateRate>10</updateRate>
+            <leftJoint>left_wheel_hinge</leftJoint>
+            <rightJoint>right_wheel_hinge</rightJoint>
+            <wheelSeparation>0.4</wheelSeparation>
+            <wheelDiameter>0.2</wheelDiameter>
+            <torque>10</torque>
+            <commandTopic>cmd_vel</commandTopic>
+            <odometryTopic>odom</odometryTopic>
+            <odometryFrame>odom</odometryFrame>
+            <robotBaseFrame>robot_footprint</robotBaseFrame>
+            <publishWheelJointState>true</publishWheelJointState>
+        </plugin>
+    </gazebo>
     <joint name="robot_footprint_joint" type="fixed">
         <origin xyz="0 0 0" rpy="0 0 0" />
@@ -61,53 +79,4 @@
         <limit effort="10000" velocity="1000"/>
         <joint_properties damping="1.0" friction="1.0"/>
-    </joint>
-    <link name='camera'>
-        <inertial>
-            <mass value="0.1"/>
-            <origin xyz="0.0 0 0" rpy=" 0 0 0"/>
-            <inertia ixx="1e-6" ixy="0" ixz="0" iyy="1e-6" iyz="0" izz="1e-6"/>
-        </inertial>
-        <collision name='camera_collision'>
-            <origin xyz="0.0 0 0" rpy=" 0 0 0"/>
-            <geometry>
-                <box size="0.05 0.05 0.05"/>
-            </geometry>
-        </collision>
-        <visual name='camera_visual'>
-            <origin xyz="0.0 0 0" rpy=" 0 0 0"/>
-            <geometry>
-                <box size="0.05 0.05 0.05"/>
-            </geometry>
-        </visual>
-    </link>
-    <joint type="fixed" name="camera_joint">
-        <origin xyz="0.2 0 0" rpy="0 0 0"/>
-        <child link="camera"/>
-        <parent link="chassis"/>
-    </joint>
-    <link name='hokuyo'>
-        <inertial>
-            <mass value="0.1"/>
-            <origin xyz="0.0 0 0" rpy=" 0 0 0"/>
-            <inertia ixx="1e-6" ixy="0" ixz="0" iyy="1e-6" iyz="0" izz="1e-6"/>
-        </inertial>
-        <collision name='hokuyo_collision'>
-            <origin xyz="0.0 0 0" rpy=" 0 0 0"/>
-            <geometry>
-                <box size="0.1 0.1 0.1"/>
-            </geometry>
-        </collision>
-        <visual name='hokuyo_visual'>
-            <origin xyz="0.0 0 0" rpy=" 0 0 0"/>
-            <geometry>
-                <mesh filename="package://bresilla/meshes/hokuyo.dae"/>
-                <!-- <box size="0.1 0.1 0.1"/> -->
-            </geometry>
-        </visual>
-    </link>
-    <joint type="fixed" name="hokuyo_joint">
-        <origin xyz="0.15 0 0.1" rpy="0 0 0"/>
-        <child link="hokuyo"/>
-        <parent link="chassis"/>
     </joint>
     <link name='chassis'>
@@ -175,3 +144,12 @@
         </visual>
     </link>
+    <gazebo reference="chassis">
+        <material>Gazebo/Blue</material>
+    </gazebo>
+    <gazebo reference="left_wheel">
+        <material>Gazebo/Green</material>
+    </gazebo>
+    <gazebo reference="right_wheel">
+        <material>Gazebo/Green</material>
+    </gazebo>
 </robot>

File: bresilla/urdf/heros_3.xacro (robot description, xacro)
@@ -1,13 +1,3 @@
 <?xml version="1.0"?>
-<!--
-Software License Agreement (BSD)
-\authors Jonathan Hechtbauer
-\maintainer Sabrina Heerklotz <sh@innok-robotics.de>
-\copyright Copyright (c) 2015, Innok Robotics GmbH, All rights reserved
-Redistribution and use in source and binary forms, with or without modification, are permitted provided that the following conditions are met:
-1. Redistributions of source code must retain the above copyright notice, this list of conditions and the following disclaimer.
-2. Redistributions in binary form must reproduce the above copyright notice, this list of conditions and the following disclaimer in the documentation and/or other materials provided with the distribution.
-THIS SOFTWARE IS PROVIDED BY THE COPYRIGHT HOLDERS AND CONTRIBUTORS "AS IS" AND ANY EXPRESS OR IMPLIED WARRANTIES, INCLUDING, BUT NOT LIMITED TO, THE IMPLIED WARRANTIES OF MERCHANTABILITY AND FITNESS FOR A PARTICULAR PURPOSE ARE DISCLAIMED. IN NO EVENT SHALL THE COPYRIGHT HOLDER OR CONTRIBUTORS BE LIABLE FOR ANY DIRECT, INDIRECT, INCIDENTAL, SPECIAL, EXEMPLARY, OR CONSEQUENTIAL DAMAGES (INCLUDING, BUT NOT LIMITED TO, PROCUREMENT OF SUBSTITUTE GOODS OR SERVICES; LOSS OF USE, DATA, OR PROFITS; OR BUSINESS INTERRUPTION) HOWEVER CAUSED AND ON ANY THEORY OF LIABILITY, WHETHER IN CONTRACT, STRICT LIABILITY, OR TORT (INCLUDING NEGLIGENCE OR OTHERWISE) ARISING IN ANY WAY OUT OF THE USE OF THIS SOFTWARE, EVEN IF ADVISED OF THE POSSIBILITY OF SUCH DAMAGE.
--->
 <robot name="innok_heros_3" xmlns:xacro="http://ros.org/wiki/xacro">
   <xacro:property name="PI" value="3.1415926535897931"/>
@@ -23,4 +13,6 @@
   <xacro:include filename="$(find bresilla)/urdf/modules/heros_battery.xacro" />
   <xacro:include filename="$(find bresilla)/urdf/modules/heros_mounting_plate.xacro" />
+  <xacro:include filename="$(find bresilla)/urdf/sensors/camera.xacro" />
+  <xacro:include filename="$(find bresilla)/urdf/sensors/hokuyo.xacro" />
   <xacro:include filename="$(find bresilla)/urdf/gazebo/heros_joint_pub.xacro" />
   <xacro:include filename="$(find bresilla)/urdf/gazebo/heros_diff_drive.xacro" />
