Commit message: added erle-rover

File: bresilla/urdf/heros_4.xacro (robot description, xacro)
@@ -1,13 +1,3 @@
 <?xml version="1.0"?>
-<!--
-Software License Agreement (BSD)
-\authors Jonathan Hechtbauer
-\maintainer Sabrina Heerklotz <sh@innok-robotics.de>
-\copyright Copyright (c) 2015, Innok Robotics GmbH, All rights reserved
-Redistribution and use in source and binary forms, with or without modification, are permitted provided that the following conditions are met:
-1. Redistributions of source code must retain the above copyright notice, this list of conditions and the following disclaimer.
-2. Redistributions in binary form must reproduce the above copyright notice, this list of conditions and the following disclaimer in the documentation and/or other materials provided with the distribution.
-THIS SOFTWARE IS PROVIDED BY THE COPYRIGHT HOLDERS AND CONTRIBUTORS "AS IS" AND ANY EXPRESS OR IMPLIED WARRANTIES, INCLUDING, BUT NOT LIMITED TO, THE IMPLIED WARRANTIES OF MERCHANTABILITY AND FITNESS FOR A PARTICULAR PURPOSE ARE DISCLAIMED. IN NO EVENT SHALL THE COPYRIGHT HOLDER OR CONTRIBUTORS BE LIABLE FOR ANY DIRECT, INDIRECT, INCIDENTAL, SPECIAL, EXEMPLARY, OR CONSEQUENTIAL DAMAGES (INCLUDING, BUT NOT LIMITED TO, PROCUREMENT OF SUBSTITUTE GOODS OR SERVICES; LOSS OF USE, DATA, OR PROFITS; OR BUSINESS INTERRUPTION) HOWEVER CAUSED AND ON ANY THEORY OF LIABILITY, WHETHER IN CONTRACT, STRICT LIABILITY, OR TORT (INCLUDING NEGLIGENCE OR OTHERWISE) ARISING IN ANY WAY OUT OF THE USE OF THIS SOFTWARE, EVEN IF ADVISED OF THE POSSIBILITY OF SUCH DAMAGE.
--->
 <robot name="innok_heros_4w" xmlns:xacro="http://ros.org/wiki/xacro">
   <xacro:property name="PI" value="3.1415926535897931"/>
@@ -21,4 +11,6 @@
   <xacro:include filename="$(find bresilla)/urdf/modules/heros_battery.xacro"/>
   <xacro:include filename="$(find bresilla)/urdf/modules/heros_mounting_plate.xacro"/>
+  <xacro:include filename="$(find bresilla)/urdf/sensors/camera.xacro" />
+  <xacro:include filename="$(find bresilla)/urdf/sensors/hokuyo.xacro" />
   <xacro:include filename="$(find bresilla)/urdf/gazebo/heros_joint_pub.xacro" />
   <xacro:include filename="$(find bresilla)/urdf/gazebo/heros_skid_drive.xacro" />

File: bresilla/urdf/modules/heros_mounting_plate.xacro (robot description, xacro)
@@ -32,5 +32,5 @@
       <origin xyz="0.46 0 -0.002" rpy="0 0 0" />
       <geometry>
-        <box size="0.92 0.72 0.004"/>
+        <box size="0.92 0.72 0"/>
       </geometry>
     </collision>

File: bresilla/urdf/modules/heros_wheel.xacro (robot description, xacro)
@@ -1,14 +1,3 @@
 <?xml version="1.0"?>
-<!--
-Description of the wheel module for the Innok Heros mobile platform.
-Software License Agreement (BSD)
-\authors Jonathan Hechtbauer
-\maintainer Sabrina Heerklotz <sh@innok-robotics.de>
-\copyright Copyright (c) 2015, Innok Robotics GmbH, All rights reserved
-Redistribution and use in source and binary forms, with or without modification, are permitted provided that the following conditions are met:
-1. Redistributions of source code must retain the above copyright notice, this list of conditions and the following disclaimer.
-2. Redistributions in binary form must reproduce the above copyright notice, this list of conditions and the following disclaimer in the documentation and/or other materials provided with the distribution.
-THIS SOFTWARE IS PROVIDED BY THE COPYRIGHT HOLDERS AND CONTRIBUTORS "AS IS" AND ANY EXPRESS OR IMPLIED WARRANTIES, INCLUDING, BUT NOT LIMITED TO, THE IMPLIED WARRANTIES OF MERCHANTABILITY AND FITNESS FOR A PARTICULAR PURPOSE ARE DISCLAIMED. IN NO EVENT SHALL THE COPYRIGHT HOLDER OR CONTRIBUTORS BE LIABLE FOR ANY DIRECT, INDIRECT, INCIDENTAL, SPECIAL, EXEMPLARY, OR CONSEQUENTIAL DAMAGES (INCLUDING, BUT NOT LIMITED TO, PROCUREMENT OF SUBSTITUTE GOODS OR SERVICES; LOSS OF USE, DATA, OR PROFITS; OR BUSINESS INTERRUPTION) HOWEVER CAUSED AND ON ANY THEORY OF LIABILITY, WHETHER IN CONTRACT, STRICT LIABILITY, OR TORT (INCLUDING NEGLIGENCE OR OTHERWISE) ARISING IN ANY WAY OUT OF THE USE OF THIS SOFTWARE, EVEN IF ADVISED OF THE POSSIBILITY OF SUCH DAMAGE.
--->
 <robot xmlns:xacro="http://ros.org/wiki/xacro" name="heros_wheel">
 <xacro:macro name="heros_wheel" params="front_rear left_right flip_y flip_z">

File: bresilla/urdf/sensors/hokuyo.xacro (robot description, xacro)
@@ -17,10 +17,9 @@
         <geometry>
           <mesh filename="package://bresilla/meshes/hokuyo.dae"/>
-          <!-- <box size="0.1 0.1 0.1"/> -->
         </geometry>
       </visual>
     </link>
     <joint type="fixed" name="hokuyo_joint">
-      <origin xyz="0.8 0 0" rpy="0 0 0"/>
+      <origin xyz="0.45 0 0.02" rpy="0 0 0"/>
       <child link="hokuyo"/>
       <parent link="mounting_plate"/>
@@ -29,5 +28,5 @@
       <sensor type="ray" name="head_hokuyo_sensor">
         <pose>0 0 0 0 0 0</pose>
-        <visualize>false</visualize>
+        <visualize>true</visualize>
         <update_rate>40</update_rate>
         <ray>
@@ -36,12 +35,12 @@
               <samples>720</samples>
               <resolution>1</resolution>
-              <min_angle>-1.570796</min_angle>
-              <max_angle>1.570796</max_angle>
+              <min_angle>-3.1570796</min_angle>
+              <max_angle>3.1570796</max_angle>
             </horizontal>
           </scan>
           <range>
             <min>0.40</min>
-            <max>30.0</max>
-            <resolution>0.02</resolution>
+            <max>20.0</max>
+            <resolution>0.01</resolution>
           </range>
           <noise>
