Commit message: write-up started

File: bresilla/urdf/modules/heros_mounting_plate.xacro (robot description, xacro)
@@ -32,5 +32,5 @@
       <origin xyz="0.46 0 -0.002" rpy="0 0 0" />
       <geometry>
-        <box size="0.92 0.72 0"/>
+        <box size="0 0 0"/>
       </geometry>
     </collision>

File: bresilla/urdf/sensors/camera.xacro (robot description, xacro)
@@ -21,7 +21,7 @@
     </link>
     <joint type="fixed" name="camera_joint">
-      <origin xyz="0.84 0 -0.02" rpy="0 0 0"/>
+      <origin xyz="0.78 0 -0.02" rpy="0 0 0"/>
       <child link="camera"/>
-      <parent link="mounting_plate"/>
+      <parent link="base_link"/>
     </joint>
     <gazebo reference="camera">

File: bresilla/urdf/sensors/hokuyo.xacro (robot description, xacro)
@@ -21,12 +21,12 @@
     </link>
     <joint type="fixed" name="hokuyo_joint">
-      <origin xyz="0.45 0 0.02" rpy="0 0 0"/>
+      <origin xyz="0.45 0 0.05" rpy="0 0 0"/>
       <child link="hokuyo"/>
-      <parent link="mounting_plate"/>
+      <parent link="base_link"/>
     </joint>
     <gazebo reference="hokuyo">
       <sensor type="ray" name="head_hokuyo_sensor">
         <pose>0 0 0 0 0 0</pose>
-        <visualize>true</visualize>
+        <visualize>false</visualize>
         <update_rate>40</update_rate>
         <ray>
@@ -35,6 +35,6 @@
               <samples>720</samples>
               <resolution>1</resolution>
-              <min_angle>-3.1570796</min_angle>
-              <max_angle>3.1570796</max_angle>
+              <min_angle>-3.570796</min_angle>
+              <max_angle>3.570796</max_angle>
             </horizontal>
           </scan>
